Commit message: Imported upstream version '0.3.0' of 'upstream'

File: franka_description/robots/panda_arm.xacro (robot description, xacro)
@@ -11,16 +11,11 @@
     <link name="${arm_id}_link0">
       <visual>
-        <origin rpy="0 0 0" xyz="0 0 0"/>
         <geometry>
-          <mesh filename="package://${description_pkg}/meshes/link0.STL"/>
+          <mesh filename="package://${description_pkg}/meshes/visual/link0.dae"/>
         </geometry>
-        <material name="">
-          <color rgba="1 1 1 1"/>
-        </material>
       </visual>
       <collision>
-        <origin rpy="0 0 0" xyz="0 0 0"/>
         <geometry>
-          <mesh filename="package://${description_pkg}/meshes/link0_collision.STL"/>
+          <mesh filename="package://${description_pkg}/meshes/collision/link0.stl"/>
         </geometry>
       </collision>
@@ -28,176 +23,141 @@
     <link name="${arm_id}_link1">
       <visual>
-        <origin rpy="0 0 0" xyz="0 0 0"/>
         <geometry>
-          <mesh filename="package://${description_pkg}/meshes/link1.STL"/>
+          <mesh filename="package://${description_pkg}/meshes/visual/link1.dae"/>
         </geometry>
-        <material name="">
-          <color rgba="1 1 1 1"/>
-        </material>
       </visual>
       <collision>
-        <origin rpy="0 0 0" xyz="0 0 0"/>
         <geometry>
-          <mesh filename="package://${description_pkg}/meshes/link1_collision.STL"/>
+          <mesh filename="package://${description_pkg}/meshes/collision/link1.stl"/>
         </geometry>
       </collision>
     </link>
     <joint name="${arm_id}_joint1" type="revolute">
-      <safety_controller k_position="100.0" k_velocity="40.0" soft_lower_limit="-2.818745" soft_upper_limit="2.818745"/>
+      <safety_controller k_position="100.0" k_velocity="40.0" soft_lower_limit="-2.8973" soft_upper_limit="2.8973"/>
       <origin rpy="0 0 0" xyz="0 0 0.333"/>
       <parent link="${arm_id}_link0"/>
       <child link="${arm_id}_link1"/>
       <axis xyz="0 0 1"/>
-      <limit effort="87" lower="-2.9671" upper="2.9671" velocity="2.5"/>
+      <limit effort="87" lower="-2.9671" upper="2.9671" velocity="2.3925"/>
     </joint>
     <link name="${arm_id}_link2">
       <visual>
-        <origin rpy="0 0 0" xyz="0 0 0"/>
         <geometry>
-          <mesh filename="package://${description_pkg}/meshes/link2.STL"/>
+          <mesh filename="package://${description_pkg}/meshes/visual/link2.dae"/>
         </geometry>
-        <material name="">
-          <color rgba="1 1 1 1"/>
-        </material>
       </visual>
       <collision>
-        <origin rpy="0 0 0" xyz="0 0 0"/>
         <geometry>
-          <mesh filename="package://${description_pkg}/meshes/link2_collision.STL"/>
+          <mesh filename="package://${description_pkg}/meshes/collision/link2.stl"/>
         </geometry>
       </collision>
     </link>
     <joint name="${arm_id}_joint2" type="revolute">
-      <safety_controller k_position="100.0" k_velocity="40.0" soft_lower_limit="-1.74097" soft_upper_limit="1.74097"/>
-      <origin rpy="-1.570796326794897 0 0" xyz="0 0 0"/>
+      <safety_controller k_position="100.0" k_velocity="40.0" soft_lower_limit="-1.7628" soft_upper_limit="1.7628"/>
+      <origin rpy="${-pi/2} 0 0" xyz="0 0 0"/>
       <parent link="${arm_id}_link1"/>
       <child link="${arm_id}_link2"/>
       <axis xyz="0 0 1"/>
-      <limit effort="87" lower="-1.8326" upper="1.8326" velocity="2.5"/>
+      <limit effort="87" lower="-1.8326" upper="1.8326" velocity="2.3925"/>
     </joint>
     <link name="${arm_id}_link3">
       <visual>
-        <origin rpy="0 0 0" xyz="0 0 0"/>
         <geometry>
-          <mesh filename="package://${description_pkg}/meshes/link3.STL"/>
+          <mesh filename="package://${description_pkg}/meshes/visual/link3.dae"/>
         </geometry>
-        <material name="">
-          <color rgba="1 1 1 1"/>
-        </material>
       </visual>
       <collision>
-        <origin rpy="0 0 0" xyz="0 0 0"/>
         <geometry>
-          <mesh filename="package://${description_pkg}/meshes/link3_collision.STL"/>
+          <mesh filename="package://${description_pkg}/meshes/collision/link3.stl"/>
         </geometry>
       </collision>
     </link>
     <joint name="${arm_id}_joint3" type="revolute">
-      <safety_controller k_position="100.0" k_velocity="40.0" soft_lower_limit="-2.818745" soft_upper_limit="2.818745"/>
-      <origin rpy="1.570796326794897 0 0" xyz="0 -0.316 0"/>
+      <safety_controller k_position="100.0" k_velocity="40.0" soft_lower_limit="-2.8973" soft_upper_limit="2.8973"/>
+      <origin rpy="${pi/2} 0 0" xyz="0 -0.316 0"/>
       <parent link="${arm_id}_link2"/>
       <child link="${arm_id}_link3"/>
       <axis xyz="0 0 1"/>
-      <limit effort="87" lower="-2.9671" upper="2.9671" velocity="2.5"/>
+      <limit effort="87" lower="-2.9671" upper="2.9671" velocity="2.3925"/>
     </joint>
     <link name="${arm_id}_link4">
       <visual>
-        <origin rpy="0 0 0" xyz="0 0 0"/>
         <geometry>
-          <mesh filename="package://${description_pkg}/meshes/link4.STL"/>
+          <mesh filename="package://${description_pkg}/meshes/visual/link4.dae"/>
         </geometry>
-        <material name="">
-          <color rgba="1 1 1 1"/>
-        </material>
       </visual>
       <collision>
-        <origin rpy="0 0 0" xyz="0 0 0"/>
         <geometry>
-          <mesh filename="package://${description_pkg}/meshes/link4_collision.STL"/>
+          <mesh filename="package://${description_pkg}/meshes/collision/link4.stl"/>
         </geometry>
       </collision>
     </link>
     <joint name="${arm_id}_joint4" type="revolute">
-      <safety_controller k_position="100.0" k_velocity="40.0" soft_lower_limit="-2.98452" soft_upper_limit="0.082935"/>
-      <origin rpy="1.570796326794897 0 0" xyz="0.0825 0 0"/>
+      <safety_controller k_position="100.0" k_velocity="40.0" soft_lower_limit="-3.0718" soft_upper_limit="0.0175"/>
+      <origin rpy="${pi/2} 0 0" xyz="0.0825 0 0"/>
       <parent link="${arm_id}_link3"/>
       <child link="${arm_id}_link4"/>
       <axis xyz="0 0 1"/>
-      <limit effort="87" lower="-3.1416" upper="0.0873" velocity="2.5"/>
+      <limit effort="87" lower="-3.1416" upper="0.0873" velocity="2.3925"/>
     </joint>
     <link name="${arm_id}_link5">
       <visual>
-        <origin rpy="0 0 0" xyz="0 0 0"/>
         <geometry>
-          <mesh filename="package://${description_pkg}/meshes/link5.STL"/>
+          <mesh filename="package://${description_pkg}/meshes/visual/link5.dae"/>
         </geometry>
-        <material name="">
-          <color rgba="1 1 1 1"/>
-        </material>
       </visual>
       <collision>
-        <origin rpy="0 0 0" xyz="0 0 0"/>
         <geometry>
-          <mesh filename="package://${description_pkg}/meshes/link5_collision.STL"/>
+          <mesh filename="package://${description_pkg}/meshes/collision/link5.stl"/>
         </geometry>
       </collision>
     </link>
     <joint name="${arm_id}_joint5" type="revolute">
-      <safety_controller k_position="100.0" k_velocity="40.0" soft_lower_limit="-2.818745" soft_upper_limit="2.818745"/>
-      <origin rpy="-1.570796326794897 0 0" xyz="-0.0825 0.384 0"/>
+      <safety_controller k_position="100.0" k_velocity="40.0" soft_lower_limit="-2.8973" soft_upper_limit="2.8973"/>
+      <origin rpy="${-pi/2} 0 0" xyz="-0.0825 0.384 0"/>
       <parent link="${arm_id}_link4"/>
       <child link="${arm_id}_link5"/>
       <axis xyz="0 0 1"/>
-      <limit effort="12" lower="-2.9671" upper="2.9671" velocity="3"/>
+      <limit effort="12" lower="-2.9671" upper="2.9671" velocity="2.8710"/>
     </joint>
     <link name="${arm_id}_link6">
       <visual>
-        <origin rpy="0 0 0" xyz="0 0 0"/>
         <geometry>
-          <mesh filename="package://${description_pkg}/meshes/link6.STL"/>
+          <mesh filename="package://${description_pkg}/meshes/visual/link6.dae"/>
         </geometry>
-        <material name="">
-          <color rgba="1 1 1 1"/>
-        </material>
       </visual>
       <collision>
-        <origin rpy="0 0 0" xyz="0 0 0"/>
         <geometry>
-          <mesh filename="package://${description_pkg}/meshes/link6_collision.STL"/>
+          <mesh filename="package://${description_pkg}/meshes/collision/link6.stl"/>
         </geometry>
       </collision>
     </link>
     <joint name="${arm_id}_joint6" type="revolute">
-      <safety_controller k_position="100.0" k_velocity="40.0" soft_lower_limit="-0.082935" soft_upper_limit="3.631185"/>
-      <origin rpy="1.570796326794897 0 0" xyz="0 0 0"/>
+      <safety_controller k_position="100.0" k_velocity="40.0" soft_lower_limit="-0.0175" soft_upper_limit="3.7525"/>
+      <origin rpy="${pi/2} 0 0" xyz="0 0 0"/>
       <parent link="${arm_id}_link5"/>
       <child link="${arm_id}_link6"/>
       <axis xyz="0 0 1"/>
-      <limit effort="12" lower="-0.0873" upper="3.8223" velocity="3"/>
+      <limit effort="12" lower="-0.0873" upper="3.8223" velocity="2.8710"/>
     </joint>
     <link name="${arm_id}_link7">
       <visual>
-        <origin rpy="0 0 0" xyz="0 0 0"/>
         <geometry>
-          <mesh filename="package://${description_pkg}/meshes/link7.STL"/>
+          <mesh filename="package://${description_pkg}/meshes/visual/link7.dae"/>
         </geometry>
-        <material name="">
-          <color rgba="1 1 1 1"/>
-        </material>
       </visual>
       <collision>
-        <origin rpy="0 0 0" xyz="0 0 0"/>
         <geometry>
-          <mesh filename="package://${description_pkg}/meshes/link7_collision.STL"/>
+          <mesh filename="package://${description_pkg}/meshes/collision/link7.stl"/>
         </geometry>
       </collision>
     </link>
     <joint name="${arm_id}_joint7" type="revolute">
-      <safety_controller k_position="100.0" k_velocity="40.0" soft_lower_limit="-2.818745" soft_upper_limit="2.818745"/>
-      <origin rpy="1.570796326794897 0 0" xyz="0.088 0 0"/>
+      <safety_controller k_position="100.0" k_velocity="40.0" soft_lower_limit="-2.8973" soft_upper_limit="2.8973"/>
+      <origin rpy="${pi/2} 0 0" xyz="0.088 0 0"/>
       <parent link="${arm_id}_link6"/>
       <child link="${arm_id}_link7"/>
       <axis xyz="0 0 1"/>
-      <limit effort="12" lower="-2.9671" upper="2.9671" velocity="3"/>
+      <limit effort="12" lower="-2.9671" upper="2.9671" velocity="2.8710"/>
     </joint>
     <link name="${arm_id}_link8"/>
